File: Drivers.kicad_sch (KiCad schematic)
At the start: 38 parts

Commit message: adjustments
Other:
- sheet Phase Driver A ports: added V_{MOTOR}; removed V_{DRV}
- sheet Phase Driver B ports: added V_{MOTOR}; removed V_{DRV}
- sheet Phase Driver C ports: added V_{MOTOR}; removed V_{DRV}
Changed lines of the file:
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@@
-			)
-		)
-		(pin "V_{DRV}" input
-			(at 195.58 115.57 180)
-			(effects
-				(font
-					(size 1.27 1.27)
-				)
-				(justify left)
 			)
 		)
@@
 				)
 				(justify right)
+			)
+		)
+		(pin "V_{MOTOR}" input
+			(at 195.58 115.57 180)
+			(effects
+				(font
+					(size 1.27 1.27)
+				)
+				(justify left)
 			)
 		)
@@
 			)
 		)
-		(pin "V_{DRV}" input
-			(at 195.58 52.07 180)
-			(effects
-				(font
-					(size 1.27 1.27)
-				)
-				(justify left)
-			)
-		)
 		(pin "LOW" input
 			(at 195.58 62.23 180)
@@
 				)
 				(justify right)
+			)
+		)
+		(pin "V_{MOTOR}" input
+			(at 195.58 52.07 180)
+			(effects
+				(font
+					(size 1.27 1.27)
+				)
+				(justify left)
 			)
 		)
@@
 			)
 		)
-		(pin "V_{DRV}" input
-			(at 195.58 83.82 180)
-			(effects
-				(font
-					(size 1.27 1.27)
-				)
-				(justify left)
-			)
-		)
 		(pin "LOW" input
 			(at 195.58 93.98 180)
@@
 			)
 		)
+		(pin "V_{MOTOR}" input
+			(at 195.58 83.82 180)
+			(effects
+				(font
+					(size 1.27 1.27)
+				)
+				(justify left)
+			)
+		)
