File: GateDriver.kicad_sch (KiCad schematic)
At the start: 10 parts, among them U2 LM1205

Commit message: adjustments
Parts:
- removed D13, D16: 5V, OpenMD:D_0402_1005Metric, symbol OpenMD:D_TVS_Small
- removed R7, R8: 0, OpenMD:R_0402_1005Metric, symbol OpenMD:R_US
- U2: value LM1205 -> UP1966E
Connections:
- net LGL is gone; now on net LOW_GATE: U2.A1 (LGL)
- net UGL is gone; now on net HIGH_GATE: U2.D1 (UGL)
- net LGH: no longer names the net of R6.1, U2.B1 (LGH)
Other:
- note added: "Substitute with LT8418, same Footprint"
- note removed: "Substitute withh UP1966 or LT8418, same Footprint"
- moved on the sheet: R6
