File: ISense.kicad_sch (KiCad schematic)
At the start: 7 parts, among them U8 INA241A2

Commit message: adjustments
Parts:
- C49: value 10nF -> 100nF
Other:
- note added: "Differential Low Pass at 80 kHz"
- note removed: "Differential Low Pass at 800 kHz"
Changed lines of the file:
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@@
 		)
 	)
-	(text "Differential Low Pass at 800 kHz"
+	(text "Differential Low Pass at 80 kHz"
 		(exclude_from_sim no)
 		(at 94.234 50.038 0)
@@
 			)
 		)
-		(property "Value" "10nF"
+		(property "Value" "100nF"
 			(at 106.6863 58.42 90)
 			(effects
