File: OpenMD.kicad_pcb (KiCad board)
At the start: 8 copper layers, 72 x 50 mm, 220 parts, among them J1 GND, J2 Digital, J3 Analog, J5 A, J6 B, J7 C, J8 V_{MOTOR}, Q1 EPC2361, Q2 EPC2361, Q3 EPC2361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

Commit message: adjustments
Parts:
- removed D12, D13, D14, D15, D16, D17: 5V, OpenMD:D_0402_1005Metric
- removed D27, D28, D29, D30, D31, D32: 6V, OpenMD:D_SOD-882
- removed R12, R13, R2, R3, R7, R8: 0, OpenMD:R_0402_1005Metric
- added C124: 1uF, OpenMD:C_0805_2012Metric, B.Cu at (127.8, 88.2)
- added C125: 1uF, OpenMD:C_0805_2012Metric, B.Cu at (129.5, 88.2)
- added C126: 1uF, OpenMD:C_0805_2012Metric, B.Cu at (127.8, 103.3)
- added C127: 1uF, OpenMD:C_0805_2012Metric, B.Cu at (129.5, 103.3)
- added C128: 1uF, OpenMD:C_0805_2012Metric, B.Cu at (127.9, 118.0)
- added C129: 1uF, OpenMD:C_0805_2012Metric, B.Cu at (129.6, 118.0)
- C28, C29, C31, C32, C34, C35: value 10uF -> 1uF; footprint OpenMD:C_1210_3225Metric -> OpenMD:C_0805_2012Metric
- C49, C54, C59: value 10nF -> 100nF
- U1, U2, U3: value LM1205 -> UP1966E
- moved G*** 30.2 mm to (125.1, 83.3)
- moved SYM1 24.0 mm to (123.6, 122.1)
- moved C88 12.8 mm to (140.3, 81.3), turned to 90 degrees
- moved C32 11.4 mm to (131.2, 88.2), turned to -90 degrees
- moved C31 2.00 mm to (131.3, 118.0)
- moved C29 1.90 mm to (131.2, 103.3)
- moved R4 1.51 mm to (132.5, 85.7)
- moved R9 1.41 mm to (132.6, 100.8)
- moved R14 1.30 mm to (132.6, 115.4)
- moved C35 0.80 mm to (133.0, 118.0)
- moved C28 0.77 mm to (132.9, 88.2)
- moved C34 0.70 mm to (132.9, 103.3)
- moved TH1 0.16 mm to (130.6, 106.3), turned to 180 degrees
Connections:
- net /Predrivers/Gate Driver A/LGH renamed Net-(U1-LGH)
- net /Predrivers/Gate Driver B/LGH renamed Net-(U2-LGH)
- net /Predrivers/Gate Driver C/LGH renamed Net-(U3-LGH)
- U1 pad A1: /Predrivers/Gate Driver A/LGL -> /AL
- U1 pad D1: /Predrivers/Gate Driver A/UGL -> /AH
- U2 pad A1: /Predrivers/Gate Driver B/LGL -> /BL
- U2 pad D1: /Predrivers/Gate Driver B/UGL -> /BH
- U3 pad A1: /Predrivers/Gate Driver C/LGL -> /CL
- U3 pad D1: /Predrivers/Gate Driver C/UGL -> /CH
Routing:
- net /V_{DRV}: track 77.9 -> 128.3 mm, vias 4 -> 3
- net /I_SENSE.A: track 79.2 -> 122.4 mm
- net /I_SENSE.C: track 108.9 -> 87.5 mm
- net /V_{MOTOR}: track 29.7 -> 46.3 mm, vias 621 -> 349
- net /I_SENSE.B: track 93.2 -> 105.5 mm
- net /SW.A: track 11.7 -> 5.37 mm, vias 97 -> 55
- net /SW.C: track 10.1 -> 5.63 mm, vias 96 -> 55
- net /SW.B: track 10.1 -> 5.66 mm, vias 94 -> 55
- net /INPUT.CL: track 37.1 -> 33.0 mm, vias 2 -> 1
- net /INPUT.CH: track 36.6 -> 33.7 mm, vias 2 -> 1
- net /INPUT.BL: track 36.9 -> 34.2 mm, vias 2 -> 1
- net /DRV_TEMP_SENSE: track 41.5 -> 39.0 mm
- net /INPUT.BH: track 36.1 -> 33.9 mm, vias 2 -> 1
- net /V_{ANA}: track 158.3 -> 156.5 mm
- net /C: track 7.78 -> 6.46 mm, vias 116 -> 12
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- removed copper zone on In1.Cu, net /A
- removed copper zone on In2.Cu, net /A
- removed copper zone on In3.Cu, net /A
- removed copper zone on In4.Cu, net /A
- removed copper zone on In1.Cu, net /B
- removed copper zone on In2.Cu, net /B
- removed copper zone on In3.Cu, net /B
- removed copper zone on In4.Cu, net /B
- removed copper zone on In1.Cu, net /C
- removed copper zone on In2.Cu, net /C
- removed copper zone on In3.Cu, net /C
- removed copper zone on In4.Cu, net /C
- removed copper zone on In2.Cu, net /GND
- removed copper zone on In6.Cu, net /GND
- removed copper zone on F.Cu, net /Predrivers/Gate Driver A/LGL
- removed copper zone on F.Cu, net /Predrivers/Gate Driver A/UGL
- removed copper zone on F.Cu, net /Predrivers/Gate Driver B/LGL
- removed copper zone on F.Cu, net /Predrivers/Gate Driver B/UGL
- removed copper zone on F.Cu, net /Predrivers/Gate Driver C/LGL
- removed copper zone on F.Cu, net /Predrivers/Gate Driver C/UGL
- removed copper zone on In2.Cu, net /SW.A
- removed copper zone on In3.Cu, net /SW.A
- removed copper zone on In4.Cu, net /SW.A
- removed copper zone on In2.Cu, net /SW.B
- removed copper zone on In3.Cu, net /SW.B
- removed copper zone on In4.Cu, net /SW.B
- removed copper zone on In2.Cu, net /SW.C
- removed copper zone on In3.Cu, net /SW.C
- removed copper zone on In4.Cu, net /SW.C
- removed copper zone on In1.Cu, net /V_{MOTOR}
- removed copper zone on In3.Cu, net /V_{MOTOR}
- removed copper zone on In5.Cu, net /V_{MOTOR}
Other:
- copper layers 8 -> 6
- board text added: "Crab Labs"
- board text added: "OpenMD Rev. ${REVISION}"
- board text added: "V_{MOTOR}"
- board text removed: "V_{BATT}"
