File: OpenMD.kicad_sch (KiCad schematic)
At the start: 27 parts, among them J1 GND, J2 Digital, J3 Analog, J5 A, J6 B, J7 C, J8 V_{MOTOR}

Commit message: adjustments
Other:
- sheet Predrivers ports: added V_{DD}; removed V_{DRV}
- note added: "Theoretical System Ratings: V_{MOTOR}: 6-80V I_{MOTOR}: 0-73A RMS P_{MAX}: 4 kW"
- note added: "V_{SENSE} = V_{MOTOR} / 25"
- note removed: "Theoretical System Ratings: V_{BATT}: 6-80V I_{BATT}: 0-73A RMS P_{MAX}: 4 kW"
- note removed: "V_{SENSE} = V_{BATT} / 25"
Changed lines of the file:
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@@
 		)
 	)
-	(text "V_{SENSE} = V_{BATT} / 25\n"
+	(text "V_{SENSE} = V_{MOTOR} / 25\n"
 		(exclude_from_sim no)
 		(at 116.078 88.392 0)
@@
 		)
 	)
-	(text "Theoretical System Ratings:\nV_{BATT}: 6-80V\nI_{BATT}: 0-73A RMS\nP_{MAX}: 4 kW"
+	(text "Theoretical System Ratings:\nV_{MOTOR}: 6-80V\nI_{MOTOR}: 0-73A RMS\nP_{MAX}: 4 kW"
 		(exclude_from_sim no)
 		(at 175.768 168.148 0)
@@
 			)
 		)
-		(pin "V_{DRV}" input
-			(at 138.43 111.76 180)
-			(effects
-				(font
-					(size 1.27 1.27)
-				)
-				(justify left)
-			)
-		)
 		(pin "GND" passive
 			(at 138.43 133.35 180)
@@
 			)
 		)
+		(pin "V_{DD}" input
+			(at 138.43 111.76 180)
+			(effects
+				(font
+					(size 1.27 1.27)
+				)
+				(justify left)
+			)
+		)
