File: PhaseDriver.kicad_sch (KiCad schematic)
At the start: 24 parts, among them Q3 EPC2361, Q6 EPC2361

Commit message: adjustments
Parts:
- removed D29, D32: 6V, OpenMD:D_SOD-882, symbol OpenMD:D_Zener_Small_Filled
- added C128, C129: 1uF, OpenMD:C_0805_2012Metric, symbol OpenMD:C
- C31, C35: value 10uF -> 1uF; footprint OpenMD:C_1210_3225Metric -> OpenMD:C_0805_2012Metric
Connections:
- net GND: now also C128.2, C129.2
- net V_{DRV} renamed V_{MOTOR}
- net V_{MOTOR}: now also C128.1, C129.1
Other:
- note added: "Medium Frequency Caps"
- note removed: "Low/Medium Frequency Caps"
- moved on the sheet: C111, C114, C117, C120, C123, C13, C17, C31, C35, C36, C55, C58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
