File: Predrivers.kicad_sch (KiCad schematic)
At the start: 0 parts

Commit message: adjustments
Changed lines of the file:
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@@
 		)
 	)
-	(hierarchical_label "V_{DRV}"
+	(hierarchical_label "V_{DD}"
 		(shape input)
 		(at 125.73 85.09 180)
@@
 		)
 	)
-	(hierarchical_label "V_{DRV}"
+	(hierarchical_label "V_{DD}"
 		(shape input)
 		(at 125.73 120.65 180)
@@
 		)
 	)
-	(hierarchical_label "V_{DRV}"
+	(hierarchical_label "V_{DD}"
 		(shape input)
 		(at 125.73 48.26 180)
